File: ortho.kicad_pcb (KiCad board)
At the start: 2 copper layers, 417.3 x 120.6 mm, 0 parts

Commit message: ortho layout schematic
made room for the controller
Parts:
- added ${REFERENCE}: SW_Gateron_LowProfile_HotSwap_PTH_rgb, my-footprints:SW_Gateron_LowProfile_HotSwap_PTH_rgb, F.Cu at (426.7, 128.7)
- added ${REFERENCE}: SW_Gateron_LowProfile_HotSwap_PTH_rgb, my-footprints:SW_Gateron_LowProfile_HotSwap_PTH_rgb, F.Cu at (426.7, 109.7)
- added ${REFERENCE}: SW_Gateron_LowProfile_HotSwap_PTH_rgb, my-footprints:SW_Gateron_LowProfile_HotSwap_PTH_rgb, F.Cu at (154.7, 185.7)
- added ${REFERENCE}: SW_Gateron_LowProfile_HotSwap_PTH_rgb, my-footprints:SW_Gateron_LowProfile_HotSwap_PTH_rgb, F.Cu at (350.7, 128.7)
- added ${REFERENCE}: SW_Gateron_LowProfile_HotSwap_PTH_rgb, my-footprints:SW_Gateron_LowProfile_HotSwap_PTH_rgb, F.Cu at (198.7, 128.7)
- added ${REFERENCE}: SW_Gateron_LowProfile_HotSwap_PTH_rgb, my-footprints:SW_Gateron_LowProfile_HotSwap_PTH_rgb, F.Cu at (110.7, 128.7)
- added ${REFERENCE}: SW_Gateron_LowProfile_HotSwap_PTH_rgb, my-footprints:SW_Gateron_LowProfile_HotSwap_PTH_rgb, F.Cu at (369.7, 185.7)
- added ${REFERENCE}: SW_Gateron_LowProfile_HotSwap_PTH_rgb, my-footprints:SW_Gateron_LowProfile_HotSwap_PTH_rgb, F.Cu at (217.7, 128.7)
- added ${REFERENCE}: SW_Gateron_LowProfile_HotSwap_PTH_rgb, my-footprints:SW_Gateron_LowProfile_HotSwap_PTH_rgb, F.Cu at (198.7, 90.7)
- added ${REFERENCE}: SW_Gateron_LowProfile_HotSwap_PTH_rgb, my-footprints:SW_Gateron_LowProfile_HotSwap_PTH_rgb, F.Cu at (255.7, 166.7)
- added ${REFERENCE}: SW_Gateron_LowProfile_HotSwap_PTH_rgb, my-footprints:SW_Gateron_LowProfile_HotSwap_PTH_rgb, F.Cu at (369.7, 147.7)
- added ${REFERENCE}: SW_Gateron_LowProfile_HotSwap_PTH_rgb, my-footprints:SW_Gateron_LowProfile_HotSwap_PTH_rgb, F.Cu at (312.7, 166.7)
- added ${REFERENCE}: SW_Gateron_LowProfile_HotSwap_PTH_rgb, my-footprints:SW_Gateron_LowProfile_HotSwap_PTH_rgb, F.Cu at (350.7, 185.7)
- added ${REFERENCE}: SW_Gateron_LowProfile_HotSwap_PTH_rgb, my-footprints:SW_Gateron_LowProfile_HotSwap_PTH_rgb, F.Cu at (217.7, 109.7)
- added ${REFERENCE}: SW_Gateron_LowProfile_HotSwap_PTH_rgb, my-footprints:SW_Gateron_LowProfile_HotSwap_PTH_rgb, F.Cu at (331.7, 185.7)
- added ${REFERENCE}: SW_Gateron_LowProfile_HotSwap_PTH_rgb, my-footprints:SW_Gateron_LowProfile_HotSwap_PTH_rgb, F.Cu at (91.8, 147.7)
- added ${REFERENCE}: SW_Gateron_LowProfile_HotSwap_PTH_rgb, my-footprints:SW_Gateron_LowProfile_HotSwap_PTH_rgb, F.Cu at (350.7, 90.7)
- added ${REFERENCE}: SW_Gateron_LowProfile_HotSwap_PTH_rgb, my-footprints:SW_Gateron_LowProfile_HotSwap_PTH_rgb, F.Cu at (331.7, 166.7)
- added ${REFERENCE}: SW_Gateron_LowProfile_HotSwap_PTH_rgb, my-footprints:SW_Gateron_LowProfile_HotSwap_PTH_rgb, F.Cu at (236.7, 128.7)
- added ${REFERENCE}: SW_Gateron_LowProfile_HotSwap_PTH_rgb, my-footprints:SW_Gateron_LowProfile_HotSwap_PTH_rgb, F.Cu at (407.7, 147.7)
- added ${REFERENCE}: SW_Gateron_LowProfile_HotSwap_PTH_rgb, my-footprints:SW_Gateron_LowProfile_HotSwap_PTH_rgb, F.Cu at (198.7, 147.7)
- added ${REFERENCE}: SW_Gateron_LowProfile_HotSwap_PTH_rgb, my-footprints:SW_Gateron_LowProfile_HotSwap_PTH_rgb, F.Cu at (154.7, 90.7)
- added ${REFERENCE}: SW_Gateron_LowProfile_HotSwap_PTH_rgb, my-footprints:SW_Gateron_LowProfile_HotSwap_PTH_rgb, F.Cu at (312.7, 147.7)
- added ${REFERENCE}: SW_Gateron_LowProfile_HotSwap_PTH_rgb, my-footprints:SW_Gateron_LowProfile_HotSwap_PTH_rgb, F.Cu at (388.7, 166.7)
- added ${REFERENCE}: SW_Gateron_LowProfile_HotSwap_PTH_rgb, my-footprints:SW_Gateron_LowProfile_HotSwap_PTH_rgb, F.Cu at (53.7, 109.7)
- added ${REFERENCE}: SW_Gateron_LowProfile_HotSwap_PTH_rgb, my-footprints:SW_Gateron_LowProfile_HotSwap_PTH_rgb, F.Cu at (293.7, 166.7)
- added ${REFERENCE}: SW_Gateron_LowProfile_HotSwap_PTH_rgb, my-footprints:SW_Gateron_LowProfile_HotSwap_PTH_rgb, F.Cu at (274.7, 185.7)
- added ${REFERENCE}: SW_Gateron_LowProfile_HotSwap_PTH_rgb, my-footprints:SW_Gateron_LowProfile_HotSwap_PTH_rgb, F.Cu at (72.8, 167.0)
- added ${REFERENCE}: SW_Gateron_LowProfile_HotSwap_PTH_rgb, my-footprints:SW_Gateron_LowProfile_HotSwap_PTH_rgb, F.Cu at (91.7, 128.5)
- added ${REFERENCE}: SW_Gateron_LowProfile_HotSwap_PTH_rgb, my-footprints:SW_Gateron_LowProfile_HotSwap_PTH_rgb, F.Cu at (255.7, 147.7)
- added ${REFERENCE}: SW_Gateron_LowProfile_HotSwap_PTH_rgb, my-footprints:SW_Gateron_LowProfile_HotSwap_PTH_rgb, F.Cu at (173.7, 185.7)
- added ${REFERENCE}: SW_Gateron_LowProfile_HotSwap_PTH_rgb, my-footprints:SW_Gateron_LowProfile_HotSwap_PTH_rgb, F.Cu at (350.7, 166.7)
- added ${REFERENCE}: SW_Gateron_LowProfile_HotSwap_PTH_rgb, my-footprints:SW_Gateron_LowProfile_HotSwap_PTH_rgb, F.Cu at (53.7, 128.7)
- added ${REFERENCE}: SW_Gateron_LowProfile_HotSwap_PTH_rgb, my-footprints:SW_Gateron_LowProfile_HotSwap_PTH_rgb, F.Cu at (173.7, 90.7)
- added ${REFERENCE}: SW_Gateron_LowProfile_HotSwap_PTH_rgb, my-footprints:SW_Gateron_LowProfile_HotSwap_PTH_rgb, F.Cu at (154.7, 128.7)
- added ${REFERENCE}: SW_Gateron_LowProfile_HotSwap_PTH_rgb, my-footprints:SW_Gateron_LowProfile_HotSwap_PTH_rgb, F.Cu at (293.7, 185.7)
- added ${REFERENCE}: SW_Gateron_LowProfile_HotSwap_PTH_rgb, my-footprints:SW_Gateron_LowProfile_HotSwap_PTH_rgb, F.Cu at (388.7, 109.7)
- added ${REFERENCE}: SW_Gateron_LowProfile_HotSwap_PTH_rgb, my-footprints:SW_Gateron_LowProfile_HotSwap_PTH_rgb, F.Cu at (369.7, 128.7)
- added ${REFERENCE}: SW_Gateron_LowProfile_HotSwap_PTH_rgb, my-footprints:SW_Gateron_LowProfile_HotSwap_PTH_rgb, F.Cu at (312.7, 185.7)
- added ${REFERENCE}: SW_Gateron_LowProfile_HotSwap_PTH_rgb, my-footprints:SW_Gateron_LowProfile_HotSwap_PTH_rgb, F.Cu at (274.7, 128.7)
- added ${REFERENCE}: SW_Gateron_LowProfile_HotSwap_PTH_rgb, my-footprints:SW_Gateron_LowProfile_HotSwap_PTH_rgb, F.Cu at (369.7, 166.7)
- added ${REFERENCE}: SW_Gateron_LowProfile_HotSwap_PTH_rgb, my-footprints:SW_Gateron_LowProfile_HotSwap_PTH_rgb, F.Cu at (407.7, 90.7)
- added ${REFERENCE}: SW_Gateron_LowProfile_HotSwap_PTH_rgb, my-footprints:SW_Gateron_LowProfile_HotSwap_PTH_rgb, F.Cu at (274.7, 109.7)
- added ${REFERENCE}: SW_Gateron_LowProfile_HotSwap_PTH_rgb, my-footprints:SW_Gateron_LowProfile_HotSwap_PTH_rgb, F.Cu at (426.7, 147.7)
- added ${REFERENCE}: SW_Gateron_LowProfile_HotSwap_PTH_rgb, my-footprints:SW_Gateron_LowProfile_HotSwap_PTH_rgb, F.Cu at (217.7, 90.7)
- added ${REFERENCE}: SW_Gateron_LowProfile_HotSwap_PTH_rgb, my-footprints:SW_Gateron_LowProfile_HotSwap_PTH_rgb, F.Cu at (91.7, 90.5)
- added ${REFERENCE}: SW_Gateron_LowProfile_HotSwap_PTH_rgb, my-footprints:SW_Gateron_LowProfile_HotSwap_PTH_rgb, F.Cu at (173.7, 128.7)
- added ${REFERENCE}: SW_Gateron_LowProfile_HotSwap_PTH_rgb, my-footprints:SW_Gateron_LowProfile_HotSwap_PTH_rgb, F.Cu at (255.7, 90.7)
- added ${REFERENCE}: SW_Gateron_LowProfile_HotSwap_PTH_rgb, my-footprints:SW_Gateron_LowProfile_HotSwap_PTH_rgb, F.Cu at (312.7, 90.7)
- added ${REFERENCE}: SW_Gateron_LowProfile_HotSwap_PTH_rgb, my-footprints:SW_Gateron_LowProfile_HotSwap_PTH_rgb, F.Cu at (255.7, 185.7)
- added ${REFERENCE}: SW_Gateron_LowProfile_HotSwap_PTH_rgb, my-footprints:SW_Gateron_LowProfile_HotSwap_PTH_rgb, F.Cu at (198.7, 109.7)
- added ${REFERENCE}: SW_Gateron_LowProfile_HotSwap_PTH_rgb, my-footprints:SW_Gateron_LowProfile_HotSwap_PTH_rgb, F.Cu at (293.7, 90.7)
- added ${REFERENCE}: SW_Gateron_LowProfile_HotSwap_PTH_rgb, my-footprints:SW_Gateron_LowProfile_HotSwap_PTH_rgb, F.Cu at (388.7, 147.7)
- added ${REFERENCE}: SW_Gateron_LowProfile_HotSwap_PTH_rgb, my-footprints:SW_Gateron_LowProfile_HotSwap_PTH_rgb, F.Cu at (53.7, 90.7)
- added ${REFERENCE}: SW_Gateron_LowProfile_HotSwap_PTH_rgb, my-footprints:SW_Gateron_LowProfile_HotSwap_PTH_rgb, F.Cu at (331.7, 128.7)
- added ${REFERENCE}: SW_Gateron_LowProfile_HotSwap_PTH_rgb, my-footprints:SW_Gateron_LowProfile_HotSwap_PTH_rgb, F.Cu at (331.7, 109.7)
- added ${REFERENCE}: SW_Gateron_LowProfile_HotSwap_PTH_rgb, my-footprints:SW_Gateron_LowProfile_HotSwap_PTH_rgb, F.Cu at (331.7, 147.7)
- added ${REFERENCE}: SW_Gateron_LowProfile_HotSwap_PTH_rgb, my-footprints:SW_Gateron_LowProfile_HotSwap_PTH_rgb, F.Cu at (72.7, 109.7)
- added ${REFERENCE}: SW_Gateron_LowProfile_HotSwap_PTH_rgb, my-footprints:SW_Gateron_LowProfile_HotSwap_PTH_rgb, F.Cu at (312.7, 128.7)
- added ${REFERENCE}: SW_Gateron_LowProfile_HotSwap_PTH_rgb, my-footprints:SW_Gateron_LowProfile_HotSwap_PTH_rgb, F.Cu at (426.7, 90.7)
- added ${REFERENCE}: SW_Gateron_LowProfile_HotSwap_PTH_rgb, my-footprints:SW_Gateron_LowProfile_HotSwap_PTH_rgb, F.Cu at (217.7, 166.7)
- added ${REFERENCE}: SW_Gateron_LowProfile_HotSwap_PTH_rgb, my-footprints:SW_Gateron_LowProfile_HotSwap_PTH_rgb, F.Cu at (198.7, 185.7)
- added ${REFERENCE}: SW_Gateron_LowProfile_HotSwap_PTH_rgb, my-footprints:SW_Gateron_LowProfile_HotSwap_PTH_rgb, F.Cu at (407.7, 166.7)
- added ${REFERENCE}: SW_Gateron_LowProfile_HotSwap_PTH_rgb, my-footprints:SW_Gateron_LowProfile_HotSwap_PTH_rgb, F.Cu at (293.7, 109.7)
- added ${REFERENCE}: SW_Gateron_LowProfile_HotSwap_PTH_rgb, my-footprints:SW_Gateron_LowProfile_HotSwap_PTH_rgb, F.Cu at (407.7, 185.7)
- added ${REFERENCE}: SW_Gateron_LowProfile_HotSwap_PTH_rgb, my-footprints:SW_Gateron_LowProfile_HotSwap_PTH_rgb, F.Cu at (350.7, 147.7)
- added ${REFERENCE}: SW_Gateron_LowProfile_HotSwap_PTH_rgb, my-footprints:SW_Gateron_LowProfile_HotSwap_PTH_rgb, F.Cu at (173.7, 109.7)
- added ${REFERENCE}: SW_Gateron_LowProfile_HotSwap_PTH_rgb, my-footprints:SW_Gateron_LowProfile_HotSwap_PTH_rgb, F.Cu at (350.7, 109.7)
- added ${REFERENCE}: SW_Gateron_LowProfile_HotSwap_PTH_rgb, my-footprints:SW_Gateron_LowProfile_HotSwap_PTH_rgb, F.Cu at (407.7, 109.7)
- added ${REFERENCE}: SW_Gateron_LowProfile_HotSwap_PTH_rgb, my-footprints:SW_Gateron_LowProfile_HotSwap_PTH_rgb, F.Cu at (110.7, 90.7)
- added ${REFERENCE}: SW_Gateron_LowProfile_HotSwap_PTH_rgb, my-footprints:SW_Gateron_LowProfile_HotSwap_PTH_rgb, F.Cu at (388.7, 185.7)
- added ${REFERENCE}: SW_Gateron_LowProfile_HotSwap_PTH_rgb, my-footprints:SW_Gateron_LowProfile_HotSwap_PTH_rgb, F.Cu at (154.7, 166.7)
- added ${REFERENCE}: SW_Gateron_LowProfile_HotSwap_PTH_rgb, my-footprints:SW_Gateron_LowProfile_HotSwap_PTH_rgb, F.Cu at (236.7, 185.7)
- added ${REFERENCE}: SW_Gateron_LowProfile_HotSwap_PTH_rgb, my-footprints:SW_Gateron_LowProfile_HotSwap_PTH_rgb, F.Cu at (293.7, 128.7)
- added ${REFERENCE}: SW_Gateron_LowProfile_HotSwap_PTH_rgb, my-footprints:SW_Gateron_LowProfile_HotSwap_PTH_rgb, F.Cu at (110.7, 166.7)
- added ${REFERENCE}: SW_Gateron_LowProfile_HotSwap_PTH_rgb, my-footprints:SW_Gateron_LowProfile_HotSwap_PTH_rgb, F.Cu at (255.7, 128.7)
- added ${REFERENCE}: SW_Gateron_LowProfile_HotSwap_PTH_rgb, my-footprints:SW_Gateron_LowProfile_HotSwap_PTH_rgb, F.Cu at (72.7, 128.7)
- added ${REFERENCE}: SW_Gateron_LowProfile_HotSwap_PTH_rgb, my-footprints:SW_Gateron_LowProfile_HotSwap_PTH_rgb, F.Cu at (217.7, 185.7)
- added ${REFERENCE}: SW_Gateron_LowProfile_HotSwap_PTH_rgb, my-footprints:SW_Gateron_LowProfile_HotSwap_PTH_rgb, F.Cu at (91.8, 166.7)
- added ${REFERENCE}: SW_Gateron_LowProfile_HotSwap_PTH_rgb, my-footprints:SW_Gateron_LowProfile_HotSwap_PTH_rgb, F.Cu at (236.7, 90.7)
- added ${REFERENCE}: SW_Gateron_LowProfile_HotSwap_PTH_rgb, my-footprints:SW_Gateron_LowProfile_HotSwap_PTH_rgb, F.Cu at (110.7, 109.7)
- added ${REFERENCE}: SW_Gateron_LowProfile_HotSwap_PTH_rgb, my-footprints:SW_Gateron_LowProfile_HotSwap_PTH_rgb, F.Cu at (72.8, 148.0)
- added ${REFERENCE}: SW_Gateron_LowProfile_HotSwap_PTH_rgb, my-footprints:SW_Gateron_LowProfile_HotSwap_PTH_rgb, F.Cu at (154.7, 109.7)
- added ${REFERENCE}: SW_Gateron_LowProfile_HotSwap_PTH_rgb, my-footprints:SW_Gateron_LowProfile_HotSwap_PTH_rgb, F.Cu at (236.7, 147.7)
- added ${REFERENCE}: SW_Gateron_LowProfile_HotSwap_PTH_rgb, my-footprints:SW_Gateron_LowProfile_HotSwap_PTH_rgb, F.Cu at (312.7, 109.7)
- added ${REFERENCE}: SW_Gateron_LowProfile_HotSwap_PTH_rgb, my-footprints:SW_Gateron_LowProfile_HotSwap_PTH_rgb, F.Cu at (91.7, 185.7)
- added ${REFERENCE}: SW_Gateron_LowProfile_HotSwap_PTH_rgb, my-footprints:SW_Gateron_LowProfile_HotSwap_PTH_rgb, F.Cu at (445.7, 109.7)
- added ${REFERENCE}: SW_Gateron_LowProfile_HotSwap_PTH_rgb, my-footprints:SW_Gateron_LowProfile_HotSwap_PTH_rgb, F.Cu at (91.7, 109.5)
- added ${REFERENCE}: SW_Gateron_LowProfile_HotSwap_PTH_rgb, my-footprints:SW_Gateron_LowProfile_HotSwap_PTH_rgb, F.Cu at (72.7, 90.7)
- added ${REFERENCE}: SW_Gateron_LowProfile_HotSwap_PTH_rgb, my-footprints:SW_Gateron_LowProfile_HotSwap_PTH_rgb, F.Cu at (53.8, 167.0)
- added ${REFERENCE}: SW_Gateron_LowProfile_HotSwap_PTH_rgb, my-footprints:SW_Gateron_LowProfile_HotSwap_PTH_rgb, F.Cu at (236.7, 109.7)
- added ${REFERENCE}: SW_Gateron_LowProfile_HotSwap_PTH_rgb, my-footprints:SW_Gateron_LowProfile_HotSwap_PTH_rgb, F.Cu at (135.7, 90.7)
- added ${REFERENCE}: SW_Gateron_LowProfile_HotSwap_PTH_rgb, my-footprints:SW_Gateron_LowProfile_HotSwap_PTH_rgb, F.Cu at (293.7, 147.7)
- added ${REFERENCE}: SW_Gateron_LowProfile_HotSwap_PTH_rgb, my-footprints:SW_Gateron_LowProfile_HotSwap_PTH_rgb, F.Cu at (135.7, 185.7)
- added ${REFERENCE}: SW_Gateron_LowProfile_HotSwap_PTH_rgb, my-footprints:SW_Gateron_LowProfile_HotSwap_PTH_rgb, F.Cu at (369.7, 109.7)
- added ${REFERENCE}: SW_Gateron_LowProfile_HotSwap_PTH_rgb, my-footprints:SW_Gateron_LowProfile_HotSwap_PTH_rgb, F.Cu at (388.7, 128.7)
- added ${REFERENCE}: SW_Gateron_LowProfile_HotSwap_PTH_rgb, my-footprints:SW_Gateron_LowProfile_HotSwap_PTH_rgb, F.Cu at (255.7, 109.7)
- added ${REFERENCE}: SW_Gateron_LowProfile_HotSwap_PTH_rgb, my-footprints:SW_Gateron_LowProfile_HotSwap_PTH_rgb, F.Cu at (331.7, 90.7)
- added ${REFERENCE}: SW_Gateron_LowProfile_HotSwap_PTH_rgb, my-footprints:SW_Gateron_LowProfile_HotSwap_PTH_rgb, F.Cu at (274.7, 90.7)
- added ${REFERENCE}: SW_Gateron_LowProfile_HotSwap_PTH_rgb, my-footprints:SW_Gateron_LowProfile_HotSwap_PTH_rgb, F.Cu at (53.8, 148.0)
- added ${REFERENCE}: SW_Gateron_LowProfile_HotSwap_PTH_rgb, my-footprints:SW_Gateron_LowProfile_HotSwap_PTH_rgb, F.Cu at (388.7, 90.7)
- added ${REFERENCE}: SW_Gateron_LowProfile_HotSwap_PTH_rgb, my-footprints:SW_Gateron_LowProfile_HotSwap_PTH_rgb, F.Cu at (217.7, 147.7)
- added ${REFERENCE}: SW_Gateron_LowProfile_HotSwap_PTH_rgb, my-footprints:SW_Gateron_LowProfile_HotSwap_PTH_rgb, F.Cu at (445.7, 128.7)
- added ${REFERENCE}: SW_Gateron_LowProfile_HotSwap_PTH_rgb, my-footprints:SW_Gateron_LowProfile_HotSwap_PTH_rgb, F.Cu at (236.7, 166.7)
- added ${REFERENCE}: SW_Gateron_LowProfile_HotSwap_PTH_rgb, my-footprints:SW_Gateron_LowProfile_HotSwap_PTH_rgb, F.Cu at (274.7, 166.7)
- added ${REFERENCE}: SW_Gateron_LowProfile_HotSwap_PTH_rgb, my-footprints:SW_Gateron_LowProfile_HotSwap_PTH_rgb, F.Cu at (135.7, 109.7)
- added ${REFERENCE}: SW_Gateron_LowProfile_HotSwap_PTH_rgb, my-footprints:SW_Gateron_LowProfile_HotSwap_PTH_rgb, F.Cu at (135.7, 128.7)
- added ${REFERENCE}: SW_Gateron_LowProfile_HotSwap_PTH_rgb, my-footprints:SW_Gateron_LowProfile_HotSwap_PTH_rgb, F.Cu at (426.7, 185.7)
- added ${REFERENCE}: SW_Gateron_LowProfile_HotSwap_PTH_rgb, my-footprints:SW_Gateron_LowProfile_HotSwap_PTH_rgb, F.Cu at (274.7, 147.7)
- added ${REFERENCE}: SW_Gateron_LowProfile_HotSwap_PTH_rgb, my-footprints:SW_Gateron_LowProfile_HotSwap_PTH_rgb, F.Cu at (407.7, 128.7)
- added ${REFERENCE}: SW_Gateron_LowProfile_HotSwap_PTH_rgb, my-footprints:SW_Gateron_LowProfile_HotSwap_PTH_rgb, F.Cu at (198.7, 166.7)
- added ${REFERENCE}: SW_Gateron_LowProfile_HotSwap_PTH_rgb, my-footprints:SW_Gateron_LowProfile_HotSwap_PTH_rgb, F.Cu at (369.7, 90.7)
- added ${REFERENCE}: SW_Gateron_LowProfile_HotSwap_PTH_rgb, my-footprints:SW_Gateron_LowProfile_HotSwap_PTH_rgb, F.Cu at (53.7, 185.7)
- added D1: , ComboDiode, F.Cu at (53.7, 195.3)
- added D10: , ComboDiode, F.Cu at (72.7, 119.3)
- added D100: , ComboDiode, F.Cu at (388.7, 100.3)
- added D101: , ComboDiode, F.Cu at (407.7, 195.3)
- added D102: , ComboDiode, F.Cu at (407.7, 176.3)
- added D103: , ComboDiode, F.Cu at (407.7, 157.3)
- added D104: , ComboDiode, F.Cu at (407.7, 138.3)
- added D105: , ComboDiode, F.Cu at (407.7, 119.3)
- added D106: , ComboDiode, F.Cu at (407.7, 100.3)
- added D107: , ComboDiode, F.Cu at (426.7, 195.3)
- added D108: , ComboDiode, F.Cu at (426.7, 157.3)
- added D109: , ComboDiode, F.Cu at (426.7, 138.3)
- added D11: , ComboDiode, F.Cu at (72.7, 100.3)
- added D110: , ComboDiode, F.Cu at (426.7, 119.3)
- added D111: , ComboDiode, F.Cu at (426.7, 100.3)
- added D112: , ComboDiode, F.Cu at (445.7, 138.3)
- added D113: , ComboDiode, F.Cu at (445.7, 119.3)
- added D12: , ComboDiode, F.Cu at (91.7, 195.3)
- added D13: , ComboDiode, F.Cu at (91.7, 176.3)
- added D14: , ComboDiode, F.Cu at (91.7, 157.3)
- added D15: , ComboDiode, F.Cu at (91.7, 138.3)
- added D16: , ComboDiode, F.Cu at (91.7, 119.3)
- added D17: , ComboDiode, F.Cu at (91.7, 100.3)
- added D18: , ComboDiode, F.Cu at (110.7, 176.3)
- added D19: , ComboDiode, F.Cu at (110.7, 138.3)
- added D2: , ComboDiode, F.Cu at (53.7, 176.3)
- added D20: , ComboDiode, F.Cu at (110.7, 119.3)
- added D21: , ComboDiode, F.Cu at (110.7, 100.3)
- added D22: , ComboDiode, F.Cu at (135.7, 195.3)
- added D23: , ComboDiode, F.Cu at (135.7, 138.3)
- added D24: , ComboDiode, F.Cu at (135.7, 119.3)
- added D25: , ComboDiode, F.Cu at (135.7, 100.3)
- added D26: , ComboDiode, F.Cu at (154.7, 195.3)
- added D27: , ComboDiode, F.Cu at (154.7, 176.3)
- added D28: , ComboDiode, F.Cu at (154.7, 138.3)
- added D29: , ComboDiode, F.Cu at (154.7, 119.3)
- added D3: , ComboDiode, F.Cu at (53.7, 157.3)
- added D30: , ComboDiode, F.Cu at (154.7, 100.3)
- added D31: , ComboDiode, F.Cu at (173.7, 195.3)
- added D32: , ComboDiode, F.Cu at (173.7, 138.3)
- added D33: , ComboDiode, F.Cu at (173.7, 119.3)
- added D34: , ComboDiode, F.Cu at (173.7, 100.3)
- added D35: , ComboDiode, F.Cu at (198.7, 195.3)
- added D36: , ComboDiode, F.Cu at (198.7, 176.3)
- added D37: , ComboDiode, F.Cu at (198.7, 157.3)
- added D38: , ComboDiode, F.Cu at (198.7, 138.3)
- added D39: , ComboDiode, F.Cu at (198.7, 119.3)
- added D4: , ComboDiode, F.Cu at (53.7, 138.3)
- added D40: , ComboDiode, F.Cu at (198.7, 100.3)
- added D41: , ComboDiode, F.Cu at (217.7, 195.3)
- added D42: , ComboDiode, F.Cu at (217.7, 176.3)
- added D43: , ComboDiode, F.Cu at (217.7, 157.3)
- added D44: , ComboDiode, F.Cu at (217.7, 138.3)
- added D45: , ComboDiode, F.Cu at (217.7, 119.3)
- added D46: , ComboDiode, F.Cu at (217.7, 100.3)
- added D47: , ComboDiode, F.Cu at (236.7, 195.3)
- added D48: , ComboDiode, F.Cu at (236.7, 176.3)
- added D49: , ComboDiode, F.Cu at (236.7, 157.3)
- added D5: , ComboDiode, F.Cu at (53.7, 119.3)
- added D50: , ComboDiode, F.Cu at (236.7, 138.3)
- added D51: , ComboDiode, F.Cu at (236.7, 119.3)
- added D52: , ComboDiode, F.Cu at (236.7, 100.3)
- added D53: , ComboDiode, F.Cu at (255.7, 195.3)
- added D54: , ComboDiode, F.Cu at (255.7, 176.3)
- added D55: , ComboDiode, F.Cu at (255.7, 157.3)
- added D56: , ComboDiode, F.Cu at (255.7, 138.3)
- added D57: , ComboDiode, F.Cu at (255.7, 119.3)
- added D58: , ComboDiode, F.Cu at (255.7, 100.3)
- added D59: , ComboDiode, F.Cu at (274.7, 195.3)
- added D6: , ComboDiode, F.Cu at (53.7, 100.3)
- added D60: , ComboDiode, F.Cu at (274.7, 176.3)
- added D61: , ComboDiode, F.Cu at (274.7, 157.3)
- added D62: , ComboDiode, F.Cu at (274.7, 138.3)
- added D63: , ComboDiode, F.Cu at (274.7, 119.3)
- added D64: , ComboDiode, F.Cu at (274.7, 100.3)
- added D65: , ComboDiode, F.Cu at (293.7, 195.3)
- added D66: , ComboDiode, F.Cu at (293.7, 176.3)
- added D67: , ComboDiode, F.Cu at (293.7, 157.3)
- added D68: , ComboDiode, F.Cu at (293.7, 138.3)
- added D69: , ComboDiode, F.Cu at (293.7, 119.3)
- added D7: , ComboDiode, F.Cu at (72.7, 176.3)
- added D70: , ComboDiode, F.Cu at (293.7, 100.3)
- added D71: , ComboDiode, F.Cu at (312.7, 195.3)
- added D72: , ComboDiode, F.Cu at (312.7, 176.3)
- added D73: , ComboDiode, F.Cu at (312.7, 157.3)
- added D74: , ComboDiode, F.Cu at (312.7, 138.3)
- added D75: , ComboDiode, F.Cu at (312.7, 119.3)
- added D76: , ComboDiode, F.Cu at (312.7, 100.3)
- added D77: , ComboDiode, F.Cu at (331.7, 195.3)
- added D78: , ComboDiode, F.Cu at (331.7, 176.3)
- added D79: , ComboDiode, F.Cu at (331.7, 157.3)
- added D8: , ComboDiode, F.Cu at (72.7, 157.3)
- added D80: , ComboDiode, F.Cu at (331.7, 138.3)
- added D81: , ComboDiode, F.Cu at (331.7, 119.3)
- added D82: , ComboDiode, F.Cu at (331.7, 100.3)
- added D83: , ComboDiode, F.Cu at (350.7, 195.3)
- added D84: , ComboDiode, F.Cu at (350.7, 176.3)
- added D85: , ComboDiode, F.Cu at (350.7, 157.3)
- added D86: , ComboDiode, F.Cu at (350.7, 138.3)
- added D87: , ComboDiode, F.Cu at (350.7, 119.3)
- added D88: , ComboDiode, F.Cu at (350.7, 100.3)
- added D89: , ComboDiode, F.Cu at (369.7, 195.3)
- added D9: , ComboDiode, F.Cu at (72.7, 138.3)
- added D90: , ComboDiode, F.Cu at (369.7, 176.3)
- added D91: , ComboDiode, F.Cu at (369.7, 157.3)
- added D92: , ComboDiode, F.Cu at (369.7, 138.3)
- added D93: , ComboDiode, F.Cu at (369.7, 119.3)
- added D94: , ComboDiode, F.Cu at (369.7, 100.3)
- added D95: , ComboDiode, F.Cu at (388.7, 195.3)
- added D96: , ComboDiode, F.Cu at (388.7, 176.3)
- added D97: , ComboDiode, F.Cu at (388.7, 157.3)
- added D98: , ComboDiode, F.Cu at (388.7, 138.3)
- added D99: , ComboDiode, F.Cu at (388.7, 119.3)
- added REF**: RP2xxx_Stamp_XL_THT, RP2xxx_Stamp:RP2xxx_Stamp_XL_THT, F.Cu at (155.3, 59.9)
Other:
- board size 417.3 x 120.6 mm -> 417.3 x 159.6 mm

Commit message: fixed custom footprint & ran matrix traces
- fixed issue with footprint not having neopixel cutout

- fixed issue with neopixel pads being on top instead of bottom
Parts:
- moved ${REFERENCE} 0.25 mm to (91.8, 148.0)
- moved ${REFERENCE} 0.25 mm to (91.8, 128.7)
- moved ${REFERENCE} 0.25 mm to (91.8, 90.7)
- moved ${REFERENCE} 0.25 mm to (91.8, 167.0)
- moved ${REFERENCE} 0.25 mm to (91.8, 186.0)
- moved ${REFERENCE} 0.25 mm to (91.8, 109.7)
Routing:
- net (no net): track 0.00 -> 4914.9 mm
Other:
- outline, holes or cut-outs redrawn
