File: ortho.kicad_pcb (KiCad board)
At the start: 2 copper layers, 417.3 x 159.6 mm, 227 parts

Commit message: rows & columns routed
Todo: LEDs and USB
Parts:
- added REF**: Wurth-632723300011, Type-C:Wurth-632723300011-HandSoldering, F.Cu at (190.3, 41.0)
- moved REF** 0.21 mm to (155.5, 59.8)
Routing:
- net (no net): track 4914.9 -> 8896.1 mm, vias 0 -> 8
