File: old_ortho/ortho_old.kicad_pcb (KiCad board)
At the start: 2 copper layers, 417.3 x 159.6 mm, 228 parts

Commit message: fixed unlinked schematic and pcb files
Parts:
- D1, D10, D100, D101, D102, D103, D104, D105, D106, D107, D108, D109, D11, D110, D111, D112, D113, D12, D13, D14, D15, D16, D17, D18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: footprint ComboDiode -> my-footprints:diode_tht
- moved REF** 82.2 mm to (108.3, 46.1), turned to -116 degrees
Routing:
- net (no net): track 8896.1 -> 9369.2 mm, vias 8 -> 55
